File: 3DOFMDB/EAGLE FILES/3dofboard.sch (EAGLE design)
At the start: 139 parts, among them U1 DRV8312_DDW_44, U2 DRV8312_DDW_44, U3 DRV8312_DDW_44

Commit message: Shrunk it down
Squeezed the motor driving parts together to get the thing to be an inch
and a half narrower (now about 3.5 inches wide)
Parts:
- removed BIGPIC: PIC32MZXXXXEC(E/F/K)144-I/PL, PIC32:PIC32MZXXXXEC(E/F/K)144-I/PL
- added C52, C58, C59: 0.1u, ASL:CAP0805
- added POWER2: (no value), ASL:M06LOCK
- added U4: PIC32MZXXXXEC(G/H/M)100-I/PT, PIC32_100PIN:PIC32MZXXXXEC(G/H/M)100-I/PT
Connections:
- new net SCK1: U$2.SCK1, U4.EBIRDY2/RPF8/SCL3/RF8
- new net SCK2: U$3.SCK1, U4.*SQICS0/RPD4/RD4
- new net SDI1: U$2.SDI1, U4.USBID/RPF3/RF3
- new net SDI2: U$3.SDI1, U4.EBID15/ETXCLK/RPD3/PMD15/RD3
- new net SDO1: U$2.SDO1, U4.EBIRDY3/RPF2/SDA3/RF2
- new net SDO2: U$3.SDO1, U4.EBID12/ETXD2/RPD12/PMD12/RD12
- new net SS1: U$2.SS1', U4.AN33/AETXD1/RPD15/SCK6/RD15
- new net SS2: U$3.SS1', U4.EBID14/ETXEN/RPD2/PMD14/RD2
- net 12V: now also POWER.3, POWER2.3; no longer POWER.2
- net 3V3: now also C52.1, C53.1, C54.1, C55.1, C56.1, C57.1, C58.1, C59.1, POWER2.4, U4.AVDD, U4.VDD, U4.VDD_2, U4.VDD_3, U4.VDD_4, U4.VDD_5, U4.VDD_6, U4.VDD_7; no longer BIGPICA.AVDD, BIGPICA.VDD, BIGPICA.VDD_2, BIGPICA.VDD_3, BIGPICA.VDD_4, C53.2, C54.2, C55.2, C56.2, C57.2
- net 5V: now also POWER.1, POWER2.1; no longer POWER.3
- net GND: now also C52.2, C53.2, C54.2, C55.2, C56.2, C57.2, C58.2, C59.2, POWER2.5, POWER2.6, U4.AVSS, U4.VSS, U4.VSS_2, U4.VSS_3, U4.VSS_4, U4.VSS_6, U4.VSS_7, U4.VSS_8; no longer BIGPICA.AVSS, BIGPICA.VSS, BIGPICA.VSS_2, BIGPICA.VSS_3, BIGPICA.VSS_4, C53.1, C54.1, C55.1, C56.1, C57.1
- net IMESA1: now also U$2.AN3/RPI33; no longer U$2.SS1'
- net IMESA2: now also U$3.AN3/RPI33; no longer U$3.SS1'
- net SCK: now also U4.EMDIO/AEMDIO/RPD0/RTCC/INT0/RD0; no longer BIGPICA.AN9/RPB14/SCK3/RB14
- net SDI: now also U4.RPD10/SCK4/RD10; no longer BIGPICA.AN32/RPD14/RD14
- net SDO: now also U4.EMDC/AEMDC/RPD11/RD11; no longer BIGPICA.AN10/RPB15/OCFB/RB15
- net SS: now also U4.EBIA15/RPD9/PMCS2/PMA15/RD9; no longer BIGPICA.AN33/RPD15/SCK6/RD15
- net VBAT: now also POWER.2, POWER2.2; no longer POWER.1
Other:
- moved on the sheet: C53, C54, C55, C56, C57

Commit message: Almost all components
Almost everything is down and routed, going to the bathroom
Parts:
- added C60, C61, C65, C66: 10u, ASL:CAP0805
- added C62, C67: .01u, ASL:CAP0805
- added C63, C68: .1u, ASL:CAP0805
- added C64, C69: 0.47u, ASL:CAP0805
- added J1: (no value), ASL:M02LOCK
- added J2: M16DUAL_ROW, ASL:M16DUAL_ROW
- added PICKIT3: (no value), ASL:M06LOCK
- added R43: 10k, ASL:RESISTOR0805-RES
- added SL1, SL2: (no value), ASL:M04LOCK
- added U$4, U$5: DRV8844PWP, drv88xx:DRV8844PWP
Connections:
- new net A10: J2.4, U4.VREF+/CVREF+/AN28/AERXD3/RA10
- new net A9: J2.3, U4.VREF-/CVREF-/AN27/AERXD2/RA9
- new net B11: J2.8, U4.AN6/ERXERR/AETXERR/RB11
- new net B12: J2.11, U4.EBIA11/AN7/ERXD0/AECRS/PMA11/RB12
- new net B13: J2.12, U4.AN8/ERXD1/AECOL/RB13
- new net B1A_EN: U$4.EN1, U4.EBID10/ETXD0/RPF1/PMD10/RF1
- new net B1A_IN: U$4.IN1, U4.EBID11/ETXD1/RPF0/PMD11/RF0
- new net B1A_OUT: SL1.1, U$4.OUT1
- new net B1B_EN: U$4.EN2, U4.EBID8/RPG0/PMD8/RG0
- new net B1B_IN: U$4.IN2, U4.EBID9/ETXERR/RPG1/PMD9/RG1
- new net B1B_OUT: SL1.2, U$4.OUT2
- new net B2A_EN: U$4.EN3, U4.EBID4/AN18/PMD4/RE4
- new net B2A_IN: U$4.IN3, U4.EBID3/RPE3/PMD3/RE3
- new net B2A_OUT: SL1.3, U$4.OUT3
- new net B2B_EN: U$4.EN4, U4.EBID6/AN16/PMD6/RE6
- new net B2B_IN: U$4.IN4, U4.EBID5/AN17/RPE5/PMD5/RE5
- new net B2B_OUT: SL1.4, U$4.OUT4
- new net B3A_EN: U$5.EN1, U4.AN14/C1IND/ECOL/RPG6/SCK2/RG6
- new net B3A_IN: U$5.IN1, U4.*EBIOE/AN19/RPC4/PMRD/RC4
- new net B3A_OUT: SL2.1, U$5.OUT1
- new net B3B_EN: U$5.EN2, U4.EBIA3/AN12/C2IND/ERXDV/ECRSDV/AERXDV/AECRSDV/RPG8/SCL4/PMA3/RG8
- new net B3B_IN: U$5.IN2, U4.EBIA4/AN13/C1INC/ECRS/RPG7/SDA4/PMA4/RG7
- new net B3B_OUT: SL2.2, U$5.OUT2
- new net B4A_EN: U$5.EN3, U4.TMS/EBIA16/AN24/RA0
- new net B4A_IN: U$5.IN3, U4.EBIA2/AN11/C2INC/ERXCLK/EREFCLK/AERXCLK/AEREFCLK/RPG9/PMA2/RG9
- new net B4A_OUT: SL2.3, U$5.OUT3
- new net B4B_EN: U$5.EN4, U4.AN26/AERXD1/RPE9/RE9, U4.PGEC2/AN46/RPB6/RB6
- new net B4B_IN: U$5.IN4, U4.AN25/AERXD0/RPE8/RE8
- new net B4B_OUT: SL2.4, U$5.OUT4
- new net CP1: C62.1, U$4.CP1
- new net CP1_1: C67.1, U$5.CP1
- new net CP2: C62.2, U$4.CP2
- new net CP2_1: C67.2, U$5.CP2
- new net FAULT_8844_1: U$4.NFAULT, U4.EBID7/AN15/PMD7/RE7
- new net FAULT_8844_2: U$5.NFAULT, U4.AN4/C1INB/RB4
- new net MCLR_BP: PICKIT3.1, R43.1, U4.*MCLR
- new net N$31: C69.1, U$5.V3P3OUT
- new net N$38: U4.AN45/C1INA/RPB5/RB5
- new net N$60: C64.1, U$4.V3P3OUT
- new net PGC_BP: PICKIT3.5, U4.PGEC1/AN1/RPB1/RB1
- new net PGD_BP: PICKIT3.4, U4.PGED1/AN0/RPB0/RB0
- new net RESET_8844_1: U$4.NRESET, U4.EBIA12/AN21/RPC2/PMA12/RC2
- new net RESET_8844_2: U$5.NRESET, U4.AN2/C2INB/RPB2/RB2
- new net RPB10: J2.7, U4.EBIA13/CVREFOUT/AN5/RPB10/PMA13/RB10
- new net RPB14: J2.13, U4.EBIA1/AN9/ERXD2/AETXD3/RPB14/SCK3/PMA1/RB14
- new net RPB15: J2.14, U4.EBIA0/AN10/ERXD3/AETXD2/RPB15/OCFB/PMA0/RB15
- new net RPB7: J2.2, U4.PGED2/AN47/RPB7/RB7
- new net RPB8: J2.5, U4.EBIA10/AN48/RPB8/PMA10/RB8
- new net RPB9: J2.6, U4.EBIA7/AN49/RPB9/PMA7/RB9
- new net RPD14: J2.16, U4.AN32/AETXD0/RPD14/RD14
- new net RPF12: J2.10, U4.TDO/EBIA17/AN31/RPF12/RF12
- new net RPF13: J2.9, U4.TDI/EBIA18/AN30/RPF13/SCK5/RF13
- new net SLEEP_8844_1: U$4.NSLEEP, U4.EBIA6/AN22/RPC1/PMA6/RC1
- new net SLEEP_8844_2: U$5.NSLEEP, U4.AN3/C2INA/RPB3/RB3
- new net VCP: C63.2, U$4.VCP
- new net VCP1: C68.2, U$5.VCP
- net 3V3: now also PICKIT3.2, R43.2
- net GND: now also C60.2, C61.2, C64.2, C65.2, C66.2, C69.2, J1.1, J2.1, J2.15, PICKIT3.3, U$4.LGND, U$4.PPAD, U$4.VNEG, U$4.VNEG1, U$4.VNEG2, U$4.VNEG3, U$5.LGND, U$5.PPAD, U$5.VNEG, U$5.VNEG1, U$5.VNEG2, U$5.VNEG3, U4.VSS_5
- net VBAT: now also C60.1, C61.1, C63.1, C65.1, C66.1, C68.1, J1.2, U$4.VM, U$4.VM1, U$5.VM, U$5.VM1

Commit message: All components placed and routed
All components placed and routed, many DRC errors, but mostly to do with
the vias on the bottom of the DRV. Need to fix those, and make sure to
put in a bunch of ground plane vias
Parts:
- added R44: 75k, ASL:RESISTOR0805-RES
- added R45: 25k, ASL:RESISTOR0805-RES
Connections:
- new net BAT_MEAS_BP: R44.2, R45.1, U4.*EBIWE/AN20/RPC3/PMWR/RC3
- net GND: now also R45.2
- net VBAT: now also R44.1
Changed lines of the file:
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@@
 <part name="PICKIT3" library="ASL" deviceset="M06" device="LOCK"/>
 <part name="R43" library="ASL" deviceset="RESISTOR" device="0805-RES" value="10k"/>
+<part name="R44" library="ASL" deviceset="RESISTOR" device="0805-RES" value="75k"/>
+<part name="R45" library="ASL" deviceset="RESISTOR" device="0805-RES" value="25k"/>
 </parts>
 <sheets>
@@
 <instance part="PICKIT3" gate="G$1" x="-482.6" y="-38.1"/>
 <instance part="R43" gate="G$1" x="-447.04" y="-25.4" rot="R90"/>
+<instance part="R44" gate="G$1" x="-462.28" y="35.56" rot="R270"/>
+<instance part="R45" gate="G$1" x="-462.28" y="20.32" rot="R270"/>
 </instances>
 <busses>
@@
 <label x="-464.82" y="-35.56" size="1.778" layer="95"/>
 </segment>
+<segment>
+<pinref part="R45" gate="G$1" pin="2"/>
+<wire x1="-462.28" y1="15.24" x2="-462.28" y2="12.7" width="0.1524" layer="91"/>
+<label x="-462.28" y="12.7" size="1.778" layer="95"/>
+</segment>
 </net>
 <net name="3V3" class="0">
@@
 <label x="-655.32" y="-33.02" size="1.778" layer="95"/>
 </segment>
+<segment>
+<pinref part="R44" gate="G$1" pin="1"/>
+<wire x1="-462.28" y1="40.64" x2="-462.28" y2="45.72" width="0.1524" layer="91"/>
+<wire x1="-459.74" y1="45.72" x2="-462.28" y2="45.72" width="0.1524" layer="91"/>
+<label x="-462.28" y="45.72" size="1.778" layer="95"/>
+</segment>
 </net>
 <net name="AGND" class="0">
@@
 </segment>
 </net>
+<net name="BAT_MEAS_BP" class="0">
+<segment>
+<pinref part="R44" gate="G$1" pin="2"/>
+<pinref part="R45" gate="G$1" pin="1"/>
+<wire x1="-462.28" y1="30.48" x2="-462.28" y2="27.94" width="0.1524" layer="91"/>
+<wire x1="-462.28" y1="27.94" x2="-462.28" y2="25.4" width="0.1524" layer="91"/>
+<wire x1="-462.28" y1="27.94" x2="-452.12" y2="27.94" width="0.1524" layer="91"/>
+<junction x="-462.28" y="27.94"/>
+<label x="-454.66" y="30.48" size="1.778" layer="95"/>
+</segment>
+<segment>
+<pinref part="U4" gate="A" pin="*EBIWE/AN20/RPC3/PMWR/RC3"/>
+<wire x1="-414.02" y1="38.1" x2="-434.34" y2="38.1" width="0.1524" layer="91"/>
+<label x="-434.34" y="38.1" size="1.778" layer="95"/>
+</segment>
+</net>

Commit message: Improved
Minor schematic adjustments (and according routing), and 8844 polygons
fixed
Connections:
- new net RPB6: J2.2, U4.PGEC2/AN46/RPB6/RB6
- net A9: no longer J2.3
- net B4B_EN: no longer U4.PGEC2/AN46/RPB6/RB6
- net RPB7: now also J2.3; no longer J2.2
Other:
- moved on the sheet: J2
Changed lines of the file:
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@@
 <instance part="SL2" gate="G$1" x="-678.18" y="-45.72"/>
 <instance part="C69" gate="G$1" x="-528.32" y="-83.82"/>
-<instance part="J2" gate="G$1" x="-289.56" y="-132.08" rot="R90"/>
+<instance part="J2" gate="G$1" x="-312.42" y="-104.14"/>
 <instance part="PICKIT3" gate="G$1" x="-482.6" y="-38.1"/>
 <instance part="R43" gate="G$1" x="-447.04" y="-25.4" rot="R90"/>
@@
 <segment>
 <pinref part="J2" gate="G$1" pin="1"/>
-<wire x1="-307.34" y1="-121.92" x2="-307.34" y2="-111.76" width="0.1524" layer="91"/>
-<label x="-307.34" y="-114.3" size="1.778" layer="95" rot="R90"/>
+<wire x1="-302.26" y1="-86.36" x2="-292.1" y2="-86.36" width="0.1524" layer="91"/>
+<label x="-294.64" y="-86.36" size="1.778" layer="95"/>
 </segment>
 <segment>
 <pinref part="J2" gate="G$1" pin="15"/>
-<wire x1="-271.78" y1="-121.92" x2="-271.78" y2="-111.76" width="0.1524" layer="91"/>
-<label x="-271.78" y="-114.3" size="1.778" layer="95" rot="R90"/>
+<wire x1="-302.26" y1="-121.92" x2="-292.1" y2="-121.92" width="0.1524" layer="91"/>
+<label x="-294.64" y="-121.92" size="1.778" layer="95"/>
 </segment>
 <segment>
@@
 </segment>
 <segment>
-<pinref part="U4" gate="A" pin="PGEC2/AN46/RPB6/RB6"/>
-<wire x1="-414.02" y1="-7.62" x2="-421.64" y2="-7.62" width="0.1524" layer="91"/>
-<label x="-421.64" y="-7.62" size="1.778" layer="95"/>
-</segment>
-<segment>
 <pinref part="U4" gate="A" pin="AN26/AERXD1/RPE9/RE9"/>
 <wire x1="-414.02" y1="10.16" x2="-421.64" y2="10.16" width="0.1524" layer="91"/>
@@
 </segment>
 <segment>
-<pinref part="J2" gate="G$1" pin="2"/>
-<wire x1="-304.8" y1="-121.92" x2="-304.8" y2="-111.76" width="0.1524" layer="91"/>
-<label x="-304.8" y="-114.3" size="1.778" layer="95" rot="R90"/>
+<pinref part="J2" gate="G$1" pin="3"/>
+<wire x1="-302.26" y1="-91.44" x2="-292.1" y2="-91.44" width="0.1524" layer="91"/>
+<label x="-294.64" y="-91.44" size="1.778" layer="95"/>
 </segment>
 </net>
@@
 <segment>
 <pinref part="J2" gate="G$1" pin="5"/>
-<wire x1="-297.18" y1="-121.92" x2="-297.18" y2="-111.76" width="0.1524" layer="91"/>
-<label x="-297.18" y="-114.3" size="1.778" layer="95" rot="R90"/>
+<wire x1="-302.26" y1="-96.52" x2="-292.1" y2="-96.52" width="0.1524" layer="91"/>
+<label x="-294.64" y="-96.52" size="1.778" layer="95"/>
 </segment>
 </net>
@@
 <segment>
 <pinref part="J2" gate="G$1" pin="6"/>
-<wire x1="-294.64" y1="-121.92" x2="-294.64" y2="-111.76" width="0.1524" layer="91"/>
-<label x="-294.64" y="-114.3" size="1.778" layer="95" rot="R90"/>
+<wire x1="-302.26" y1="-99.06" x2="-292.1" y2="-99.06" width="0.1524" layer="91"/>
+<label x="-294.64" y="-99.06" size="1.778" layer="95"/>
 </segment>
 </net>
@@
 <segment>
 <pinref part="J2" gate="G$1" pin="7"/>
-<wire x1="-292.1" y1="-121.92" x2="-292.1" y2="-111.76" width="0.1524" layer="91"/>
-<label x="-292.1" y="-114.3" size="1.778" layer="95" rot="R90"/>
+<wire x1="-302.26" y1="-101.6" x2="-292.1" y2="-101.6" width="0.1524" layer="91"/>
+<label x="-294.64" y="-101.6" size="1.778" layer="95"/>
 </segment>
 </net>
@@
 <segment>
 <pinref part="J2" gate="G$1" pin="9"/>
-<wire x1="-287.02" y1="-121.92" x2="-287.02" y2="-111.76" width="0.1524" layer="91"/>
-<label x="-287.02" y="-114.3" size="1.778" layer="95" rot="R90"/>
+<wire x1="-302.26" y1="-106.68" x2="-292.1" y2="-106.68" width="0.1524" layer="91"/>
+<label x="-294.64" y="-106.68" size="1.778" layer="95"/>
 </segment>
 </net>
@@
 <segment>
 <pinref part="J2" gate="G$1" pin="10"/>
-<wire x1="-284.48" y1="-121.92" x2="-284.48" y2="-111.76" width="0.1524" layer="91"/>
-<label x="-284.48" y="-114.3" size="1.778" layer="95" rot="R90"/>
+<wire x1="-302.26" y1="-109.22" x2="-292.1" y2="-109.22" width="0.1524" layer="91"/>
+<label x="-294.64" y="-109.22" size="1.778" layer="95"/>
 </segment>
 </net>
@@
 <segment>
 <pinref part="J2" gate="G$1" pin="13"/>
-<wire x1="-276.86" y1="-121.92" x2="-276.86" y2="-111.76" width="0.1524" layer="91"/>
-<label x="-276.86" y="-114.3" size="1.778" layer="95" rot="R90"/>
+<wire x1="-302.26" y1="-116.84" x2="-292.1" y2="-116.84" width="0.1524" layer="91"/>
+<label x="-294.64" y="-116.84" size="1.778" layer="95"/>
 </segment>
 </net>
@@
 <segment>
 <pinref part="J2" gate="G$1" pin="14"/>
-<wire x1="-274.32" y1="-121.92" x2="-274.32" y2="-111.76" width="0.1524" layer="91"/>
-<label x="-274.32" y="-114.3" size="1.778" layer="95" rot="R90"/>
+<wire x1="-302.26" y1="-119.38" x2="-292.1" y2="-119.38" width="0.1524" layer="91"/>
+<label x="-294.64" y="-119.38" size="1.778" layer="95"/>
 </segment>
 </net>
@@
 <segment>
 <pinref part="J2" gate="G$1" pin="16"/>
-<wire x1="-269.24" y1="-121.92" x2="-269.24" y2="-111.76" width="0.1524" layer="91"/>
-<label x="-269.24" y="-114.3" size="1.778" layer="95" rot="R90"/>
+<wire x1="-302.26" y1="-124.46" x2="-292.1" y2="-124.46" width="0.1524" layer="91"/>
+<label x="-294.64" y="-124.46" size="1.778" layer="95"/>
 </segment>
 </net>
@@
 <label x="-421.64" y="-12.7" size="1.778" layer="95"/>
 </segment>
-<segment>
-<pinref part="J2" gate="G$1" pin="3"/>
-<wire x1="-302.26" y1="-121.92" x2="-302.26" y2="-111.76" width="0.1524" layer="91"/>
-<label x="-302.26" y="-114.3" size="1.778" layer="95" rot="R90"/>
-</segment>
 </net>
 <net name="A10" class="0">
@@
 <segment>
 <pinref part="J2" gate="G$1" pin="4"/>
-<wire x1="-299.72" y1="-121.92" x2="-299.72" y2="-111.76" width="0.1524" layer="91"/>
-<label x="-299.72" y="-114.3" size="1.778" layer="95" rot="R90"/>
+<wire x1="-302.26" y1="-93.98" x2="-292.1" y2="-93.98" width="0.1524" layer="91"/>
+<label x="-294.64" y="-93.98" size="1.778" layer="95"/>
 </segment>
 </net>
@@
 <segment>
 <pinref part="J2" gate="G$1" pin="8"/>
-<wire x1="-289.56" y1="-121.92" x2="-289.56" y2="-111.76" width="0.1524" layer="91"/>
-<label x="-289.56" y="-114.3" size="1.778" layer="95" rot="R90"/>
+<wire x1="-302.26" y1="-104.14" x2="-292.1" y2="-104.14" width="0.1524" layer="91"/>
+<label x="-294.64" y="-104.14" size="1.778" layer="95"/>
 </segment>
 </net>
@@
 <segment>
 <pinref part="J2" gate="G$1" pin="11"/>
-<wire x1="-281.94" y1="-121.92" x2="-281.94" y2="-111.76" width="0.1524" layer="91"/>
-<label x="-281.94" y="-114.3" size="1.778" layer="95" rot="R90"/>
+<wire x1="-302.26" y1="-111.76" x2="-292.1" y2="-111.76" width="0.1524" layer="91"/>
+<label x="-294.64" y="-111.76" size="1.778" layer="95"/>
 </segment>
 </net>
@@
 <segment>
 <pinref part="J2" gate="G$1" pin="12"/>
-<wire x1="-279.4" y1="-121.92" x2="-279.4" y2="-111.76" width="0.1524" layer="91"/>
-<label x="-279.4" y="-114.3" size="1.778" layer="95" rot="R90"/>
+<wire x1="-302.26" y1="-114.3" x2="-292.1" y2="-114.3" width="0.1524" layer="91"/>
+<label x="-294.64" y="-114.3" size="1.778" layer="95"/>
 </segment>
 </net>
@@
 </segment>
 </net>
+<net name="RPB6" class="0">
+<segment>
+<pinref part="J2" gate="G$1" pin="2"/>
+<wire x1="-302.26" y1="-88.9" x2="-292.1" y2="-88.9" width="0.1524" layer="91"/>
+<label x="-294.64" y="-88.9" size="1.778" layer="95"/>
+</segment>
+<segment>
+<pinref part="U4" gate="A" pin="PGEC2/AN46/RPB6/RB6"/>
+<wire x1="-414.02" y1="-7.62" x2="-421.64" y2="-7.62" width="0.1524" layer="91"/>
+<label x="-421.64" y="-7.62" size="1.778" layer="95"/>
+</segment>
+</net>

Commit message: Passes DRC
Now passes DRC
Other:
- moved on the sheet: U1, U2, U3

Commit message: Names, GND vias, Mounting holes
Moved the names around so they don't overlap, added a bunch of ground
vias (not very systematically), and 4 mounting holes in the corners (not
quite symmetrical)
Parts:
- renumbered MOTOR_CONNECT to MC, MOTOR_CONNECT1 to MC1, MOTOR_CONNECT2 to MC2

Commit message: Moved the DSPIC33 library into the github repo
yup, that's it
Parts:
- U$1, U$2, U$3: device microchip:DSPIC33EP512MC502-28SSOP -> DSPIC33:DSPIC33EP512MC502-28SSOP
Changed lines of the file:
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@@
 <part name="U2" library="DRV83x2Support" deviceset="DRV8312_DDW_44" device=""/>
 <part name="CS1" library="3DOFMDB_COMPONENTS" deviceset="MAX4376" device=""/>
-<part name="U$1" library="microchip" deviceset="DSPIC33EP512MC502-28SSOP" device=""/>
+<part name="U$1" library="DSPIC33" deviceset="DSPIC33EP512MC502-28SSOP" device=""/>
 <part name="C1" library="ASL" deviceset="CAP" device="0805" value="0.1u"/>
 <part name="C2" library="ASL" deviceset="CAP" device="0805" value="0.1u"/>
@@
 <part name="U1" library="DRV83x2Support" deviceset="DRV8312_DDW_44" device=""/>
 <part name="CS2" library="3DOFMDB_COMPONENTS" deviceset="MAX4376" device=""/>
-<part name="U$2" library="microchip" deviceset="DSPIC33EP512MC502-28SSOP" device=""/>
+<part name="U$2" library="DSPIC33" deviceset="DSPIC33EP512MC502-28SSOP" device=""/>
 <part name="C18" library="ASL" deviceset="CAP" device="0805" value="0.1u"/>
 <part name="C19" library="ASL" deviceset="CAP" device="0805" value="0.1u"/>
@@
 <part name="U3" library="DRV83x2Support" deviceset="DRV8312_DDW_44" device=""/>
 <part name="CS3" library="3DOFMDB_COMPONENTS" deviceset="MAX4376" device=""/>
-<part name="U$3" library="microchip" deviceset="DSPIC33EP512MC502-28SSOP" device=""/>
+<part name="U$3" library="DSPIC33" deviceset="DSPIC33EP512MC502-28SSOP" device=""/>
 <part name="C35" library="ASL" deviceset="CAP" device="0805" value="0.1u"/>
 <part name="C36" library="ASL" deviceset="CAP" device="0805" value="0.1u"/>
